Commit message: adding launch files

File: urdf/youbot_base/base.urdf.xacro (robot description, xacro)
@@ -268,4 +268,131 @@
       </collision>
     </link>
+    <link name="camera_link">
+      <visual>
+        <geometry>
+          <box size="0.03 0.03 0.015"/> <!-- Representation of the camera -->
+        </geometry>
+        <material name="Orange"/>
+      </visual>
+    </link>
+    <joint name="joint_camera_chassis" type="fixed">
+      <parent link="base_link"/>
+      <child link="camera_link"/>
+      <origin xyz="0.05 0 0.1" rpy="0 0 0"/>
+    </joint>
+    <link name="left_camera_link">
+      <visual>
+        <geometry>
+          <box size="0.01 0.01 0.01"/> <!-- Representation of the left camera -->
+        </geometry>
+        <material name="Orange"/>
+      </visual>
+    </link>
+    <joint name="joint_left_camera" type="fixed">
+      <parent link="camera_link"/>
+      <child link="left_camera_link"/>
+      <origin xyz="0 0.02 0" rpy="-1.5707963 0 -1.5707963"/>
+    </joint>
+    <link name="right_camera_link">
+      <visual>
+        <geometry>
+          <box size="0.01 0.01 0.01"/> <!-- Representation of the right camera -->
+        </geometry>
+        <material name="Orange"/>
+      </visual>
+    </link>
+    <joint name="joint_right_camera" type="fixed">
+      <parent link="camera_link"/>
+      <child link="right_camera_link"/>
+      <origin xyz="0 -0.02 0" rpy="-1.5707963 0 -1.5707963"/>
+    </joint>
+    <gazebo reference="camera_link">
+      <sensor type="multicamera" name="stereo_camera">
+        <update_rate>10.0</update_rate>
+        <camera name="left">
+          <pose>0 0.02 0 0 0 0</pose>
+          <horizontal_fov>1.3962634</horizontal_fov>
+          <image>
+            <width>640</width>
+            <height>480</height>
+            <format>R8G8B8</format>
+          </image>
+          <clip>
+            <near>0.02</near>
+            <far>300</far>
+          </clip>
+          <noise>
+            <type>gaussian</type>
+            <mean>0.0</mean>
+            <stddev>0.007</stddev>
+          </noise>
+        </camera>
+        <camera name="right">
+          <pose>0 -0.02 0 0 0 0</pose>
+          <horizontal_fov>1.3962634</horizontal_fov>
+          <image>
+            <width>640</width>
+            <height>480</height>
+            <format>R8G8B8</format>
+          </image>
+          <clip>
+            <near>0.02</near>
+            <far>300</far>
+          </clip>
+          <noise>
+            <type>gaussian</type>
+            <mean>0.0</mean>
+            <stddev>0.007</stddev>
+          </noise>
+        </camera>
+        <plugin name="stereo_camera_controller" filename="libgazebo_ros_multicamera.so">
+          <alwaysOn>true</alwaysOn>
+          <updateRate>10.0</updateRate>
+          <cameraName>multisense_sl/camera</cameraName>
+          <imageTopicName>image_raw</imageTopicName>
+          <cameraInfoTopicName>camera_info</cameraInfoTopicName>
+          <frameName>left_camera_link</frameName>
+          <rightFrameName>right_camera_link</rightFrameName>
+          <hackBaseline>0.04</hackBaseline>
+          <distortionK1>0.0</distortionK1>
+          <distortionK2>0.0</distortionK2>
+          <distortionK3>0.0</distortionK3>
+          <distortionT1>0.0</distortionT1>
+          <distortionT2>0.0</distortionT2>
+        </plugin>
+      </sensor>
+    </gazebo>
+    <gazebo reference="base_link">
+      <gravity>true</gravity>
+      <sensor name="imu_sensor" type="imu">
+        <always_on>true</always_on>
+        <update_rate>10</update_rate>
+        <visualize>true</visualize>
+        <topic>__default_topic__</topic>
+        <plugin filename="libgazebo_ros_imu_sensor.so" name="imu_plugin">
+          <topicName>/imu/data</topicName>
+          <bodyName>base_link</bodyName>
+          <updateRateHZ>10.0</updateRateHZ>
+          <gaussianNoise>0.0</gaussianNoise>
+          <xyzOffset>0 0 0</xyzOffset>
+          <rpyOffset>0 0 0</rpyOffset>
+          <frameName>base_link</frameName>
+          <initialOrientationAsReference>false</initialOrientationAsReference>
+        </plugin>
+        <pose>0 0 0 0 0 0</pose>
+      </sensor>
+    </gazebo>
+    <link name="lidar_link">
+      <visual>
+        <geometry>
+          <box size="0.0 0.0 0.0"/> <!-- Representation of the camera -->
+        </geometry>
+      </visual>
+    </link>
+    <joint name="$joint_base_lidar" type="fixed">
+      <origin xyz="0 0 0" rpy="0 0 0"/>
+      <parent link="base_link"/>
+      <child link="lidar_link"/>
+    </joint>
     <!-- extensions -->
     <xacro:youbot_base_gazebo/>
